Commit message: Update finaltask.xacro

File: brics/finaltask_description/urdf/finaltask.xacro (robot description, xacro)
@@ -94,5 +94,5 @@
   <parent link="base_link"/>
   <child link="rightwheel_1"/>
-  <axis xyz="0.0 -1.0 0.0"/>
+  <axis xyz="0.0 1.0 0.0"/>
 </joint>
 <joint name="Rev3" type="continuous">
